File: addon-yd-esp32s3/Power Manager.kicad_sch (KiCad schematic)
At the start: 33 parts, among them Q1 Q_NMOS_DGS, Q2 Q_NMOS_DGS, Q3 DMP2160U-7, U1 DW01A, U3 TP4056, U4 TLV62565DBVR, U5 SDB628

Commit message: completando el diseño
Parts:
- removed D3: 1N5819, Diode_SMD:D_SOD-123, symbol Diode:B120-E3
- added C8: 1uF, Capacitor_SMD:C_0603_1608Metric, symbol Device:C
- added JP2: Jumper_2_Open, Jumper:SolderJumper-2_P1.3mm_Open_TrianglePad1.0x1.5mm, symbol Jumper:Jumper_2_Open
Connections:
- net GND: now also C8.2
- net VBAT: now also Q3.3 (D)
- net VBUS: now also C8.1
- net VSUP: now also Q3.2 (S), JP2.1 (A); no longer C5.1, Q3.3 (D), U4.1 (EN), U4.4 (VIN)
- new net: C5.1, JP2.2 (B), U4.1 (EN), U4.4 (VIN)
Other:
- moved on the sheet: D4, Q3, R6

Commit message: completando diseño PCB
Parts:
- removed Q2: Q_NMOS_DGS, Package_TO_SOT_SMD:SOT-23, symbol Transistor_FET:Q_NMOS_DGS
- added Q2: SI2302, Package_TO_SOT_SMD:SOT-23, symbol Transistor_FET:Q_NMOS_GSD
- B1: LCSC C2988620 -> (none); LCSC Part (none) -> C2988620; Mfr. Part (none) -> BH-18650-B1BA002; Part # BH-18650-B1BA002 -> (none)
- C8: footprint Capacitor_SMD:C_0603_1608Metric -> Capacitor_SMD:C_0805_2012Metric; symbol Device:C -> kmr:C_1uF_0805; IPN (none) -> IPN-0006; InvenTree (none) -> 5; LCSC Part (none) -> C28323; Manufacturer (none) -> Samsung Electro-Mechanics; Mfr. Part (none) -> CL21B105KBFNNNE; Part URL (none) -> http://inv.kuska-iot.com/part/5/; Price (none) -> 0.001
- Q1: value Q_NMOS_DGS -> SI2302; symbol Transistor_FET:Q_NMOS_DGS -> Transistor_FET:Q_NMOS_GSD; LCSC Part (none) -> C2891732; Manufacturer (none) -> YONGYUTAI; Mfr. Part (none) -> SI2302; Price (none) -> 0.00112
- R5, R6: symbol Device:R_US -> kmr:R_100k_0603; IPN (none) -> IPN-0013; InvenTree (none) -> 13; LCSC Part (none) -> C14675; Manufacturer (none) -> YAGEO; Mfr. Part (none) -> RC0603FR-07100KL; Part URL (none) -> http://inv.kuska-iot.com/part/13/; Price (none) -> 0.001
- U1: LCSC C351410 -> (none); LCSC Part (none) -> C351410; Mfr. Part (none) -> DW01A; Part # DW01A -> (none)
Connections:
- net GND: now also Q1.2 (S); no longer Q1.3 (S)
- net GNDV: now also Q2.2 (S)
- net at U1.1 (OD): now also Q2.1 (G)
- net at U1.3 (OC): now also Q1.1 (G); no longer Q1.2 (G)
- new net: Q1.3 (D), Q2.3 (D)
Other:
- title: (none) -> ${TITLE}

Commit message: completando version 1
Parts:
- B1: LCSC (none) -> C2988620; LCSC Part C2988620 -> (none); Mfr. Part BH-18650-B1BA002 -> (none); Part # (none) -> BH-18650-B1BA002
- C1, C5: LCSC (none) -> C1705; LCSC Part C1705 -> (none); Mfr. Part CL10A475KP8NNNC -> (none); Part # (none) -> CL10A475KP8NNNC
- C2: LCSC (none) -> C66501; LCSC Part C66501 -> (none); Mfr. Part CL10B104KO8NNNC -> (none); Part # (none) -> CL10B104KO8NNNC
- C3, C4, C7: LCSC (none) -> C5674; LCSC Part C5674 -> (none); Mfr. Part CL21A226MQQNNNE -> (none); Part # (none) -> CL21A226MQQNNNE
- C6: LCSC (none) -> C17024; LCSC Part C17024 -> (none); Mfr. Part CL21A106KPFNNNE -> (none); Part # (none) -> CL21A106KPFNNNE
- C8: LCSC (none) -> C28323; LCSC Part C28323 -> (none); Mfr. Part CL21B105KBFNNNE -> (none); Part # (none) -> CL21B105KBFNNNE
- D1: LCSC (none) -> C965804; LCSC Part C965804 -> (none); Mfr. Part XL-1608UGC-04 -> (none); Part # (none) -> XL-1608UGC-04
- D2: LCSC (none) -> C84263; LCSC Part C84263 -> (none); Mfr. Part NCD0603R1 -> (none); Part # (none) -> NCD0603R1
- D4, D5: LCSC (none) -> C82544; LCSC Part C82544 -> (none); Mfr. Part 1N5819HW-7-F -> (none); Part # (none) -> 1N5819HW-7-F
- L1: LCSC (none) -> C83472; LCSC Part C83472 -> (none); Mfr. Part SWPA4030S220MT -> (none); Part # (none) -> SWPA4030S220MT
- L2: LCSC (none) -> C86081; LCSC Part C86081 -> (none); Mfr. Part LQH44PN2R2MP0L -> (none); Part # (none) -> LQH44PN2R2MP0L
- Q1, Q2: LCSC (none) -> C2891732; LCSC Part C2891732 -> (none); Mfr. Part SI2302 -> (none); Part # (none) -> SI2302
- Q3: LCSC (none) -> C260875; LCSC Part C260875 -> (none); Mfr. Part DMP2160U-7 -> (none); Part # (none) -> DMP2160U-7
- R1, R3: LCSC (none) -> C21190; LCSC Part C21190 -> (none); Mfr. Part 0603WAF1001T5E -> (none); Part # (none) -> 0603WAF1001T5E
- R10: LCSC (none) -> C22885; LCSC Part C22885 -> (none); Mfr. Part 0603WAF1622T5E -> (none); Part # (none) -> 0603WAF1622T5E
- R11: LCSC (none) -> C4190; LCSC Part C4190 -> (none); Mfr. Part 0603WAF2201T5E -> (none); Part # (none) -> 0603WAF2201T5E
- R2: LCSC (none) -> C23179; LCSC Part C23179 -> (none); Mfr. Part 0603WAF4700T5E -> (none); Part # (none) -> 0603WAF4700T5E
- R4: LCSC (none) -> C22765; LCSC Part C22765 -> (none); Mfr. Part 0603WAF1201T5E -> (none); Part # (none) -> 0603WAF1201T5E
- R5: symbol kmr:R_100k_0603 -> kmr:R_100_0603; IPN IPN-0013 -> RES-000156-00; InvenTree 13 -> 156; LCSC (none) -> C105588; LCSC Part C14675 -> (none); Mfr. Part RC0603FR-07100KL -> (none); Part # (none) -> RC0603FR-07100RL; Part URL http://inv.kuska-iot.com/part/13/ -> http://inv.kuska-iot.com/part/156/; Rated Power (none) -> -; Temperature Range (none) -> -; Tolerance (none) -> -
- R6: LCSC (none) -> C14675; LCSC Part C14675 -> (none); Mfr. Part RC0603FR-07100KL -> (none); Part # (none) -> RC0603FR-07100KL
- R7: LCSC (none) -> C22984; LCSC Part C22984 -> (none); Mfr. Part 0603WAF3002T5E -> (none); Part # (none) -> 0603WAF3002T5E
- R8: LCSC (none) -> C23192; LCSC Part C23192 -> (none); Mfr. Part 0603WAF5103T5E -> (none); Part # (none) -> 0603WAF5103T5E
- R9: LCSC (none) -> C25808; LCSC Part C25808 -> (none); Mfr. Part 0603WAF1203T5E -> (none); Part # (none) -> 0603WAF1203T5E
- U1: LCSC (none) -> C351410; LCSC Part C351410 -> (none); Mfr. Part DW01A -> (none); Part # (none) -> DW01A
- U3: LCSC (none) -> C725790; LCSC Part C725790 -> (none); Mfr. Part TP4056 -> (none); Part # (none) -> TP4056
- U4: LCSC (none) -> C87122; LCSC Part C87122 -> (none); Mfr. Part TLV62565DBVR -> (none); Part # (none) -> TLV62565DBVR
- U5: LCSC (none) -> C77805; LCSC Part C77805 -> (none); Mfr. Part SDB628 -> (none); Part # (none) -> SDB628
