File: addon-yd-esp32s3/addon-yd-esp32s3.kicad_sch (KiCad schematic)
At the start: 4 parts, among them J1 Conn_01x22, J2 Conn_01x22, J3 Conn_01x02, J5 Conn_01x15

Commit message: completando el diseño
Parts:
- added JP1: Jumper_2_Open, Jumper:SolderJumper-2_P1.3mm_Open_TrianglePad1.0x1.5mm, symbol Jumper:Jumper_2_Open
- added TP1, TP2: TestPoint, TestPoint:TestPoint_Pad_1.5x1.5mm, symbol Connector:TestPoint
Connections:
- net +3V3: now also JP1.2 (B); no longer J1.21 (Pin_21), J1.22 (Pin_22)
- net GND: now also TP2.1
- net Power Manager/VBUS: now also TP1.1
- new net: J1.21 (Pin_21), J1.22 (Pin_22), JP1.1 (A)
Other:
- moved on the sheet: J3, J5

Commit message: completando diseño PCB
Parts:
- J2, J5: now left out of the parts list
- J3: value Conn_01x02 -> S2B-PH-K-S(LF)(SN); LCSC Part (none) -> C173752; Manufacturer (none) -> JST; Mfr. Part (none) -> S2B-PH-K-S(LF)(SN); Price (none) -> 0.034
Other:
- title: (none) -> ${TITLE}
- moved on the sheet: J3, TP1, TP2

Commit message: completando version 1
Parts:
- J3: LCSC (none) -> C173752; LCSC Part C173752 -> (none); Mfr. Part S2B-PH-K-S(LF)(SN) -> (none); Part # (none) -> S2B-PH-K-S(LF)(SN)
Connections:
- no-connect marks 0 -> 28
Changed lines of the file:
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@@
 		(color 0 0 0 0)
+	)
+	(no_connect
+		(at 254 69.85)
+	)
+	(no_connect
+		(at 220.98 82.55)
+	)
+	(no_connect
+		(at 220.98 59.69)
+	)
+	(no_connect
+		(at 220.98 46.99)
+	)
+	(no_connect
+		(at 220.98 57.15)
+	)
+	(no_connect
+		(at 220.98 72.39)
+	)
+	(no_connect
+		(at 254 87.63)
+	)
+	(no_connect
+		(at 220.98 74.93)
+	)
+	(no_connect
+		(at 254 82.55)
+	)
+	(no_connect
+		(at 254 64.77)
+	)
+	(no_connect
+		(at 254 57.15)
+	)
+	(no_connect
+		(at 220.98 54.61)
+	)
+	(no_connect
+		(at 220.98 67.31)
+	)
+	(no_connect
+		(at 220.98 77.47)
+	)
+	(no_connect
+		(at 254 54.61)
+	)
+	(no_connect
+		(at 220.98 62.23)
+	)
+	(no_connect
+		(at 220.98 87.63)
+	)
+	(no_connect
+		(at 254 67.31)
+	)
+	(no_connect
+		(at 254 74.93)
+	)
+	(no_connect
+		(at 254 90.17)
+	)
+	(no_connect
+		(at 254 77.47)
+	)
+	(no_connect
+		(at 220.98 80.01)
+	)
+	(no_connect
+		(at 254 85.09)
+	)
+	(no_connect
+		(at 220.98 90.17)
+	)
+	(no_connect
+		(at 220.98 64.77)
+	)
+	(no_connect
+		(at 220.98 85.09)
+	)
+	(no_connect
+		(at 254 72.39)
+	)
+	(no_connect
+		(at 254 80.01)
 	)
 	(wire
@@
 			)
 		)
-		(property "Part #" ""
+		(property "Part #" "S2B-PH-K-S(LF)(SN)"
 			(at 83.82 97.79 0)
 			(effects
@@
 			)
 		)
-		(property "LCSC" ""
+		(property "LCSC" "C173752"
 			(at 83.82 97.79 0)
 			(effects
@@
 			)
 		)
-		(property "LCSC Part" "C173752"
+		(property "Mfr. Part" ""
 			(at 83.82 97.79 0)
 			(effects
-				(font
-					(size 1.27 1.27)
-				)
-				(hide yes)
-			)
-		)
-		(property "Mfr. Part" "S2B-PH-K-S(LF)(SN)"
-			(at 83.82 97.79 0)
-			(effects
